Commit message: update urdf files to integrate with moveit

File: src/franka_description/urdf/panda_arm_hand.urdf (robot description, URDF)
Before this commit: robot panda, 10 links, 9 joints
Links:
- added link panda_hand, mass 5; collision mesh filename=package://franka_description/meshes/collision/hand.stl; visual mesh filename=package://franka_description/meshes/visual/hand.dae
- added link panda_leftfinger, mass 5; collision mesh filename=package://franka_description/meshes/collision/finger.stl; visual mesh filename=package://franka_description/meshes/visual/finger.dae
- added link panda_rightfinger, mass 5; collision mesh filename=package://franka_description/meshes/collision/finger.stl; visual mesh filename=package://franka_description/meshes/visual/finger.dae
Joints:
- added joint panda_finger_joint1: type prismatic, parent panda_hand, child panda_leftfinger, origin xyz=0 0 0.0584 rpy=0 0 0, axis 0 1 0, limit lower=0.0 upper=0.04 effort=20 velocity=0.2
- added joint panda_finger_joint2: type prismatic, parent panda_hand, child panda_rightfinger, origin xyz=0 0 0.0584 rpy=0 0 0, axis 0 -1 0, limit lower=0.0 upper=0.04 effort=20 velocity=0.2, mimic joint=panda_finger_joint1
- added joint panda_hand_joint: type fixed, parent panda_link8, child panda_hand, origin xyz=0 0 0 rpy=0 0 -0.785398163397
