Commit message: add/up files to be able to control robot in gazebo

File: src/franka_description/urdf/panda_arm_hand_custom.urdf (robot description, URDF)
Before this commit: robot panda, 12 links, 11 joints
Links:
- removed link panda_link8
- added link world
Joints:
- removed joint panda_joint8
- added joint fixed: type fixed, parent world, child panda_link0
- joint panda_hand_joint: parent panda_link8 -> panda_link7
